File: MECB_68008/MECB_68008_CPU.kicad_pcb (KiCad board)
At the start: 2 copper layers, 99.8 x 99.8 mm, 27 parts, among them J1 MECB_64AC, SW1 SW_DIP_PB, U1 ATF22V10C-15PU, U2 SST39SF040, U3 MC68008FN, U4 TC1232CPA, U5 GAL22V10, U6 AS6C4008-55, U7 74LS73, Y1 8 MHz

Commit message: v1.1 board finalised
Parts:
- removed C7, C8: 0.1uF, Capacitor_THT:C_Disc_D5.0mm_W2.5mm_P2.50mm
- removed the R1 at (128.0, 83.7)
- removed U7: 74LS73, Package_DIP:DIP-14_W7.62mm_LongPads
- C1, C2, C3, C4, C5, C6: footprint Capacitor_THT:C_Disc_D5.0mm_W2.5mm_P2.50mm -> Capacitor_THT:C_Disc_D5.0mm_W2.5mm_P5.00mm
- R1: renamed from R2; value 10K -> 4K7
- moved C5 48.2 mm to (118.2, 102.1)
- moved U5 48.0 mm to (116.9, 107.1)
- moved C1 47.1 mm to (118.0, 55.0)
- moved U1 46.0 mm to (116.9, 60.3)
- moved R1 42.6 mm to (169.5, 61.5)
- moved JP2 38.6 mm to (163.2, 85.2), turned to 90 degrees
- moved C6 20.1 mm to (153.0, 93.5), turned to 180 degrees
- moved U6 16.2 mm to (148.8, 98.5)
- moved U4 12.5 mm to (182.4, 82.5)
- moved U2 11.9 mm to (172.8, 98.4)
- moved C2 11.4 mm to (173.0, 93.5)
- moved C4 10.6 mm to (180.5, 77.5)
- moved Y1 10.5 mm to (181.9, 63.0)
- moved U3 3.15 mm to (133.5, 67.3)
- moved C3 2.78 mm to (137.8, 49.8)
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Connections:
- net ROM_WR renamed ROM_R~{W}
- J1 pad A14: /ECB_A19 -> ECB_A19
- J1 pad A18: /ECB_A14 -> ECB_A14
- J1 pad A27: ECB_IORQ -> ~{ECB_IORQ}
- J1 pad A29: /ECB_A13 -> ECB_A13
- J1 pad C10: /ECB_A16 -> ECB_A16
- J1 pad C12: /ECB_A17 -> ECB_A17
- J1 pad C13: /ECB_A18 -> ECB_A18
- J1 pad C19: /ECB_A21 -> ECB_A21
- J1 pad C20: ECB_NMI -> ~{ECB_NMI}
- J1 pad C21: ECB_INT -> ~{ECB_INT}
- J1 pad C22: ECB_WR -> CPU_R~{W}
- J1 pad C23: /ECB_A20 -> ECB_A20
- J1 pad C24: CPU_RW -> ~{ECB_RD}
- J1 pad C27: /ECB_A12 -> ECB_A12
- J1 pad C28: /ECB_A15 -> ECB_A15
- J1 pad C29: ECB_CLK -> E
- J1 pad C30: ECB_MREQ -> ~{ECB_MREQ}
- J1 pad C31: ECB_RESET -> ~{ECB_RESET}
- JP2 pad 1: ECB_WR -> CPU_R~{W}
- RN1 pad 2: ECB_INT -> ~{ECB_INT}
- RN1 pad 3: ECB_NMI -> ~{ECB_NMI}
- RN1 pad 4: ECB_RESET -> ~{ECB_RESET}
- RN1 pad 9: unconnected-(RN1-R8-Pad9) -> ~{DTACK}
- U1 pad 10: unconnected-(U1-IN_8-Pad10) -> CPUSP
- U1 pad 11: unconnected-(U1-IN_9-Pad11) -> ECB_A17
- U1 pad 13: unconnected-(U1-IN_10-Pad13) -> ECB_A16
- U1 pad 14: ~{IPL2} -> ECB_A15
- U1 pad 15: ~{IPL1} -> ECB_A14
- U1 pad 16: ~{IPL0} -> ECB_A13
- U1 pad 17: unconnected-(U1-I/O_4-Pad17) -> ECB_A12
- U1 pad 18: unconnected-(U1-I/O_5-Pad18) -> ~{DTACK}
- U1 pad 19: unconnected-(U1-I/O_6-Pad19) -> ~{ECB_MREQ}
- U1 pad 20: unconnected-(U1-I/O_7-Pad20) -> ~{ECB_IORQ}
- U1 pad 21: unconnected-(U1-I/O_8-Pad21) -> ~{CS_RAM}
- U1 pad 22: unconnected-(U1-I/O_9-Pad22) -> ~{CS_ROM}
- U1 pad 23: unconnected-(U1-I/O_10-Pad23) -> PPDTACK
- U1 pad 3: CPU_RW -> BOOT
- U1 pad 4: ECB_NMI -> ~{ECB_RESET}
- U1 pad 5: ECB_INT -> ECB_A21
- U1 pad 6: BOOT -> ECB_A20
- U1 pad 7: FC2 -> ECB_A19
- U1 pad 8: FC1 -> ECB_A18
- U1 pad 9: FC0 -> CPU_R~{W}
- U2 pad 1: /ECB_A18 -> ECB_A18
- U2 pad 2: /ECB_A16 -> ECB_A16
- U2 pad 22: CS_ROM -> ~{CS_ROM}
- U2 pad 24: CPU_RW -> ~{ECB_RD}
- U2 pad 28: /ECB_A13 -> ECB_A13
- U2 pad 29: /ECB_A14 -> ECB_A14
- U2 pad 3: /ECB_A15 -> ECB_A15
- U2 pad 30: /ECB_A17 -> ECB_A17
- U2 pad 4: /ECB_A12 -> ECB_A12
- U3 pad 11: /ECB_A12 -> ECB_A12
- U3 pad 12: /ECB_A13 -> ECB_A13
- U3 pad 13: /ECB_A21 -> ECB_A21
- U3 pad 14: /ECB_A14 -> ECB_A14
- U3 pad 16: /ECB_A15 -> ECB_A15
- U3 pad 18: /ECB_A16 -> ECB_A16
- U3 pad 19: /ECB_A17 -> ECB_A17
- U3 pad 20: /ECB_A18 -> ECB_A18
- U3 pad 21: /ECB_A19 -> ECB_A19
- U3 pad 22: /ECB_A20 -> ECB_A20
- U3 pad 33: CPU_RW -> CPU_R~{W}
- U3 pad 38: ECB_CLK -> SYS_CLK
- U3 pad 41: ECB_RESET -> ~{ECB_RESET}
- U3 pad 43: ~{VPA} -> ~{ECB_IORQ}
- U4 pad 7: ECB_CLK -> SYS_CLK
- U5 pad 10: /ECB_A18 -> ECB_A18
- U5 pad 11: CPU_RW -> CPU_R~{W}
- U5 pad 13: ECB_MREQ -> unconnected-(U5-I13-Pad13)
- U5 pad 16: ECB_RESET -> ~{ECB_RESET}
- U5 pad 17: IORQ -> ~{IPL2}
- U5 pad 18: CS_RAM -> ~{IPL1}
- U5 pad 19: CS_ROM -> ~{IPL0}
- U5 pad 20: ~{DTACK} -> unconnected-(U5-IO20-Pad20)
- U5 pad 22: ECB_WR -> ~{ECB_RD}
- U5 pad 23: PPDTACK -> unconnected-(U5-IO23-Pad23)
- U5 pad 7: /ECB_A21 -> ~{ECB_INT}
- U5 pad 8: /ECB_A20 -> ~{ECB_NMI}
- U5 pad 9: /ECB_A19 -> ECB_A19
- U6 pad 1: /ECB_A18 -> ECB_A18
- U6 pad 2: /ECB_A16 -> ECB_A16
- U6 pad 22: CS_RAM -> ~{CS_RAM}
- U6 pad 24: CPU_RW -> ~{ECB_RD}
- U6 pad 28: /ECB_A13 -> ECB_A13
- U6 pad 29: ECB_WR -> CPU_R~{W}
- U6 pad 3: /ECB_A14 -> ECB_A14
- U6 pad 30: /ECB_A17 -> ECB_A17
- U6 pad 31: /ECB_A15 -> ECB_A15
- U6 pad 4: /ECB_A12 -> ECB_A12
- Y1 pad 5: ECB_CLK -> SYS_CLK
Routing:
- net CPU_R~{W}: track 0.00 -> 201.3 mm, vias 0 -> 5
- net CPU_RW: track 200.5 -> 0.00 mm, vias 2 -> 0
- net ~{ECB_RESET}: track 0.00 -> 159.3 mm, vias 0 -> 4
- net ECB_WR: track 155.2 -> 0.00 mm, vias 3 -> 0
- net ECB_A18: track 0.00 -> 148.7 mm, vias 0 -> 1
- net ~{CS_ROM}: track 0.00 -> 148.3 mm, vias 0 -> 2
- net ECB_A17: track 0.00 -> 145.2 mm, vias 0 -> 1
- net ~{ECB_NMI}: track 0.00 -> 141.8 mm, vias 0 -> 2
- net ECB_A13: track 0.00 -> 140.3 mm, vias 0 -> 2
- net /ECB_A14: track 137.9 -> 0.00 mm, vias 4 -> 0
- net /ECB_A18: track 135.9 -> 0.00 mm, vias 2 -> 0
- net /ECB_A13: track 130.0 -> 0.00 mm, vias 1 -> 0
- net ECB_A14: track 0.00 -> 128.2 mm, vias 0 -> 3
- net ECB_A19: track 0.00 -> 128.1 mm, vias 0 -> 4
- net ECB_RESET: track 127.3 -> 0.00 mm, vias 4 -> 0
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Other:
- board text added: "68008 CPU Card v1.1"
- board text added: "GND"
- board text added: "RD"
- board text added: "RESET"
- board text added: "ROM WE"
- board text added: "WR"
