File: MECB_Z80/MECB_Z80_CPU/MECB_Z80_CPU.kicad_pcb (KiCad board)
At the start: 2 copper layers, 99.8 x 99.8 mm, 27 parts, among them J1 MECB_64AC, SW1 SW_DIP_PB, U1 ATF22V10C-15PU, U2 SST39SF040, U3 AS6C4008-55, U4 TC1232CPA, U5 Z84C00xxP, U6 74HC670, U7 74HC670, U8 74HC74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

Commit message: Minor fixes for v1.0
Parts:
- added J2: CLK_SEL, Connector_IDC:IDC-Header_2x03_P2.54mm_Vertical, F.Cu at (133.0, 56.9)
- moved U8 15.6 mm to (147.4, 56.9)
- moved U4 5.03 mm to (160.9, 68.0)
- moved C4 5.03 mm to (159.0, 63.0)
Connections:
- U1 pad 16: unconnected-(U1-I/O_3-Pad16) -> /~{ECB_MREQ}
- U1 pad 17: /~{ECB_MREQ} -> /~{ECB_IORQ}
- U1 pad 18: /~{ECB_IORQ} -> /CLK4
- U1 pad 19: /ECB_CLK -> /CLK2
Routing:
- net /MA17: track 219.1 -> 99.7 mm, vias 6 -> 0
- net /~{MREQ}: track 178.3 -> 88.0 mm, vias 3 -> 5
- net /ECB_D1: track 98.2 -> 179.7 mm, vias 1 -> 7
- net /ECB_A9: track 118.8 -> 193.2 mm, vias 3 -> 8
- net /~{ECB_RD}: track 167.1 -> 240.5 mm, vias 4 -> 5
- net /ECB_A13: track 124.5 -> 176.3 mm, vias 1 -> 4
- net /ECB_A4: track 205.5 -> 155.0 mm, vias 5 -> 6
- net /~{ECB_WR}: track 236.2 -> 191.8 mm, vias 4 -> 5
- net /ECB_A2: track 170.0 -> 213.7 mm, vias 4 -> 7
- net /ECB_A8: track 172.9 -> 132.5 mm, vias 5 -> 1
- net /MA14: track 93.6 -> 132.3 mm, vias 6 -> 5
- net /ECB_A10: track 124.7 -> 161.6 mm, vias 1 -> 5
- net /~{ECB_INT}: track 89.2 -> 125.1 mm, vias 2 -> 4
- net /ECB_D5: track 187.9 -> 155.7 mm, vias 3 -> 8
- net /~{ECB_WAIT}: track 71.7 -> 99.0 mm, vias 2 -> 1
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- added copper zone on F.Cu, net +5V
- added copper zone on B.Cu, net GND
- removed copper zone on B.Cu, net (none)
- removed copper zone on F.Cu, net (none)
