File: MECB_Z80/MECB_Z80_CPU/MECB_Z80_CPU.kicad_sch (KiCad schematic)
At the start: 27 parts, among them J1 MECB_64AC, SW1 SW_DIP_PB, U1 ATF22V10C-15PU, U2 SST39SF040, U3 AS6C4008-55, U4 TC1232CPA, U5 Z84C00xxP, U6 74HC670, U7 74HC670, U8 74HC74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

Commit message: Minor fixes for v1.0
Parts:
- added J2: CLK_SEL, Connector_IDC:IDC-Header_2x03_P2.54mm_Vertical, symbol Connector_Generic:Conn_02x03_Odd_Even
Connections:
- net ECB_CLK: now also J2.2 (Pin_2), J2.4 (Pin_4), J2.6 (Pin_6); no longer U1.19 (I/O_6)
- net SYS_CLK: now also J2.1 (Pin_1)
- net ~{ECB_IORQ}: now also U1.17 (I/O_4); no longer U1.18 (I/O_5)
- net ~{ECB_MREQ}: now also U1.16 (I/O_3); no longer U1.17 (I/O_4)
- new net CLK2: J2.3 (Pin_3), U1.19 (I/O_6)
- new net CLK4: J2.5 (Pin_5), U1.18 (I/O_5)
Changed lines of the file:
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@@
 	)
 	(junction
+		(at 226.06 40.64)
+		(diameter 0)
+		(color 0 0 0 0)
+	)
+	(junction
 		(at 34.29 187.96)
 		(diameter 0)
@@
 	)
 	(junction
+		(at 226.06 43.18)
+		(diameter 0)
+		(color 0 0 0 0)
+	)
+	(junction
 		(at 55.88 118.11)
 		(diameter 0)
@@
 	)
 	(junction
+		(at 166.37 27.94)
+		(diameter 0)
+		(color 0 0 0 0)
+	)
+	(junction
 		(at 71.12 105.41)
 		(diameter 0)
@@
 	(wire
 		(pts
+			(xy 200.66 48.26) (xy 209.55 48.26)
+		)
+		(stroke
+			(width 0)
+			(type default)
+		)
+	)
+	(wire
+		(pts
 			(xy 217.17 102.87) (xy 226.06 102.87)
 		)
@@
 	(wire
 		(pts
+			(xy 226.06 60.96) (xy 226.06 43.18)
+		)
+		(stroke
+			(width 0)
+			(type default)
+		)
+	)
+	(wire
+		(pts
 			(xy 109.22 144.78) (xy 109.22 146.05)
 		)
@@
 	(wire
 		(pts
-			(xy 200.66 40.64) (xy 209.55 40.64)
+			(xy 213.36 38.1) (xy 213.36 17.78)
+		)
+		(stroke
+			(width 0)
+			(type default)
+		)
+	)
+	(wire
+		(pts
+			(xy 200.66 40.64) (xy 213.36 40.64)
 		)
 		(stroke
@@
 	(wire
 		(pts
+			(xy 213.36 17.78) (xy 166.37 17.78)
+		)
+		(stroke
+			(width 0)
+			(type default)
+		)
+	)
+	(wire
+		(pts
 			(xy 106.68 81.28) (xy 116.84 81.28)
 		)
@@
 	(wire
 		(pts
+			(xy 200.66 45.72) (xy 209.55 45.72)
+		)
+		(stroke
+			(width 0)
+			(type default)
+		)
+	)
+	(wire
+		(pts
 			(xy 31.75 137.16) (xy 41.91 137.16)
 		)
@@
 	(wire
 		(pts
-			(xy 157.48 27.94) (xy 167.64 27.94)
+			(xy 157.48 27.94) (xy 166.37 27.94)
 		)
 		(stroke
@@
 	(wire
 		(pts
+			(xy 226.06 40.64) (xy 226.06 43.18)
+		)
+		(stroke
+			(width 0)
+			(type default)
+		)
+	)
+	(wire
+		(pts
 			(xy 74.93 163.83) (xy 82.55 163.83)
 		)
@@
 	(wire
 		(pts
+			(xy 166.37 27.94) (xy 167.64 27.94)
+		)
+		(stroke
+			(width 0)
+			(type default)
+		)
+	)
+	(wire
+		(pts
 			(xy 81.28 48.26) (xy 83.82 48.26)
 		)
@@
 	(wire
 		(pts
+			(xy 166.37 17.78) (xy 166.37 27.94)
+		)
+		(stroke
+			(width 0)
+			(type default)
+		)
+	)
+	(wire
+		(pts
 			(xy 31.75 30.48) (xy 34.29 30.48)
 		)
@@
 	(wire
 		(pts
-			(xy 200.66 45.72) (xy 209.55 45.72)
-		)
-		(stroke
-			(width 0)
-			(type default)
-		)
-	)
-	(wire
-		(pts
 			(xy 107.95 163.83) (xy 118.11 163.83)
 		)
@@
 	(wire
 		(pts
-			(xy 200.66 43.18) (xy 209.55 43.18)
-		)
-		(stroke
-			(width 0)
-			(type default)
-		)
-	)
-	(wire
-		(pts
 			(xy 74.93 166.37) (xy 82.55 166.37)
 		)
@@
 	(wire
 		(pts
+			(xy 226.06 38.1) (xy 226.06 40.64)
+		)
+		(stroke
+			(width 0)
+			(type default)
+		)
+	)
+	(wire
+		(pts
 			(xy 203.2 100.33) (xy 212.09 100.33)
 		)
@@
 	(wire
 		(pts
+			(xy 213.36 60.96) (xy 226.06 60.96)
+		)
+		(stroke
+			(width 0)
+			(type default)
+		)
+	)
+	(wire
+		(pts
 			(xy 203.2 128.27) (xy 212.09 128.27)
 		)
@@
 	(wire
 		(pts
+			(xy 200.66 43.18) (xy 213.36 43.18)
+		)
+		(stroke
+			(width 0)
+			(type default)
+		)
+	)
+	(wire
+		(pts
 			(xy 232.41 35.56) (xy 241.3 35.56)
 		)
@@
 		)
 	)
-	(label "~{ECB_MREQ}"
-		(at 201.93 45.72 0)
-		(effects
-			(font
-				(size 1.27 1.27)
-			)
-			(justify left bottom)
-		)
-	)
 	(label "~{ECB_M1}"
 		(at 163.83 87.63 0)
@@
 		)
 	)
+	(label "ECB_CLK"
+		(at 214.63 60.96 0)
+		(effects
+			(font
+				(size 1.27 1.27)
+			)
+			(justify left bottom)
+		)
+	)
 	(label "~{PAGE_EN}"
 		(at 73.66 186.69 0)
@@
 		)
 	)
+	(label "~{ECB_IORQ}"
+		(at 201.93 45.72 0)
+		(effects
+			(font
+				(size 1.27 1.27)
+			)
+			(justify left bottom)
+		)
+	)
 	(label "ECB_D0"
 		(at 204.47 123.19 0)
@@
 		)
 	)
+	(label "~{ECB_MREQ}"
+		(at 201.93 48.26 0)
+		(effects
+			(font
+				(size 1.27 1.27)
+			)
+			(justify left bottom)
+		)
+	)
 	(label "~{ECB_IORQ}"
 		(at 33.02 160.02 0)
@@
 		)
 	)
-	(label "~{ECB_IORQ}"
-		(at 201.93 43.18 0)
-		(effects
-			(font
-				(size 1.27 1.27)
-			)
-			(justify left bottom)
-		)
-	)
 	(label "ECB_A11"
 		(at 33.02 111.76 0)
@@
 		)
 	)
-	(label "ECB_CLK"
+	(label "CLK2"
 		(at 201.93 40.64 0)
 		(effects
@@
 		)
 	)
+	(label "CLK4"
+		(at 201.93 43.18 0)
+		(effects
+			(font
+				(size 1.27 1.27)
+			)
+			(justify left bottom)
+		)
+	)
 	(label "ECB_A6"
 		(at 201.93 53.34 0)
@@
 					(unit 1)
 				)
+			)
+		)
+	)
+	(symbol
+		(lib_id "Connector_Generic:Conn_02x03_Odd_Even")
+		(at 218.44 40.64 0)
+		(unit 1)
+		(exclude_from_sim no)
+		(in_bom yes)
+		(on_board yes)
+		(dnp no)
+		(fields_autoplaced yes)
+		(property "Reference" "J2"
+			(at 219.71 31.75 0)
+			(effects
+				(font
+					(size 1.27 1.27)
+				)
+			)
+		)
+		(property "Value" "CLK_SEL"
+			(at 219.71 34.29 0)
+			(effects
+				(font
+					(size 1.27 1.27)
+				)
+			)
+		)
+		(property "Footprint" "Connector_IDC:IDC-Header_2x03_P2.54mm_Vertical"
+			(at 218.44 40.64 0)
+			(effects
+				(font
+					(size 1.27 1.27)
+				)
+				(hide yes)
+			)
+		)
+		(property "Datasheet" "~"
+			(at 218.44 40.64 0)
+			(effects
+				(font
+					(size 1.27 1.27)
+				)
+				(hide yes)
+			)
+		)
+		(property "Description" "Generic connector, double row, 02x03, odd/even pin numbering scheme (row 1 odd numbers, row 2 even numbers), script generated (kicad-library-utils/schlib/autogen/connector/)"
+			(at 218.44 40.64 0)
+			(effects
+				(font
+					(size 1.27 1.27)
+				)
+				(hide yes)
+			)
+		)
+		(pin "1"
+		)
+		(pin "3"
+		)
+		(pin "5"
+		)
+		(pin "2"
+		)
+		(pin "4"
+		)
+		(pin "6"
+		)
+		(instances
+			(project ""
+				(path "/1a2f72d1-0b36-4610-afc4-4ad1660d5d3b"
+					(reference "J2")
+					(unit 1)
+				)
