File: MECB_8088/MECB_8088_CPU/MECB_8088_CPU.kicad_pcb (KiCad board)
At the start: 2 copper layers, 99.8 x 99.8 mm, 28 parts, among them J1 MECB_64AC, SW1 SW_DIP_PB, U1 ATF22V10C-15PU, U2 SST39SF040, U3 AS6C4008-55, U4 TC1232CPA, U5 74HCT573, U6 74HCT75, U7 8088-2, Y1 8 MHz

Commit message: v1.1 - fix for missing ECB_CLK signal
Connections:
- U1 pad 14: unconnected-(U1-I/O_1-Pad14) -> /ECB_CLK
Routing:
- net /ECB_A0: track 86.4 -> 151.4 mm, vias 1 -> 5
- net /~{CS_RAM}: track 128.8 -> 171.2 mm, vias 3 -> 2
- net /ECB_A9: track 146.8 -> 186.8 mm, vias 3 -> 2
- net /ECB_CLK: track 0.00 -> 39.2 mm, vias 0 -> 1
- net /ECB_A13: track 131.0 -> 161.3 mm, vias 1 -> 3
- net /ECB_D3: track 194.6 -> 164.5 mm, vias 4 -> 2
- net /ECB_D4: track 157.9 -> 187.1 mm
- net /ECB_A6: track 125.9 -> 97.3 mm
- net /ECB_A15: track 137.7 -> 165.1 mm
- net /ECB_A16: track 128.2 -> 154.2 mm, vias 0 -> 4
- net /~{ECB_WR}: track 119.3 -> 141.4 mm, vias 2 -> 4
- net /ECB_A4: track 107.0 -> 88.0 mm
- net /ECB_A7: track 108.8 -> 127.4 mm, vias 2 -> 3
- net /~{ECB_NMI}: track 154.6 -> 170.3 mm, vias 1 -> 3
- net /ECB_A8: track 160.2 -> 146.0 mm, vias 3 -> 4
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Other:
- board text added: "8088 CPU Card v1.1"
- board text removed: "8088 CPU Card v1.0"

Commit message: v1.1 8088 board
Parts:
- removed R1, R2, R3: 4K7, Resistor_THT:R_Axial_DIN0309_L9.0mm_D3.2mm_P12.70mm_Horizontal
- added J2: CLK_SEL, Connector_IDC:IDC-Header_2x03_P2.54mm_Vertical, F.Cu at (168.0, 66.5)
- added RN2: 4K7, Resistor_THT:R_Array_SIP9, F.Cu at (176.5, 67.9)
- RN1: value 10K -> 4K7
- moved U5 2.60 mm to (116.4, 111.5)
Connections:
- U1 pad 11: unconnected-(U1-IN_9-Pad11) -> /~{SS0}
- U1 pad 14: /ECB_CLK -> unconnected-(U1-I/O_1-Pad14)
- U1 pad 15: /HOLD -> /CLK/8
- U1 pad 16: /INT -> /CLK/4
- U1 pad 17: /NMI -> /CLK/2
- U1 pad 18: /~{ECB_RESET} -> /INT
- U1 pad 19: /~{ECB_MREQ} -> /NMI
- U1 pad 2: /~{M} -> /~{ECB_MREQ}
- U1 pad 20: /~{ECB_IORQ} -> /~{ECB_RESET}
- U1 pad 21: /~{CS_RAM} -> /~{ECB_IORQ}
- U1 pad 22: /~{CS_ROM} -> /~{CS_RAM}
- U1 pad 23: /~{TEST} -> /~{CS_ROM}
- U1 pad 8: /RESET -> /HOLD
- U4 pad 5: /RESET -> /HOLD
- U5 pad 1: /RESET -> /HOLD
- U7 pad 21: /RESET -> /HOLD
- U7 pad 28: /~{M} -> /~{ECB_MREQ}
- U7 pad 34: unconnected-(U7-~{SSO}-Pad34) -> /~{SS0}
Routing:
- net /HOLD: track 25.5 -> 154.7 mm, vias 0 -> 2
- net /RESET: track 122.1 -> 0.00 mm, vias 4 -> 0
- net /~{ECB_NMI}: track 170.3 -> 93.1 mm, vias 3 -> 0
- net /ECB_CLK: track 39.2 -> 107.9 mm
- net /CLK/8: track 0.00 -> 63.9 mm, vias 0 -> 1
- net /ECB_A16: track 154.2 -> 217.8 mm
- net /~{SS0}: track 0.00 -> 58.9 mm, vias 0 -> 3
- net /CLK/4: track 0.00 -> 51.8 mm
- net /~{M}: track 50.8 -> 0.00 mm, vias 2 -> 0
- net /CLK/2: track 0.00 -> 50.0 mm
- net /ECB_A0: track 151.4 -> 101.5 mm, vias 5 -> 3
- net /~{CS_RAM}: track 171.2 -> 126.3 mm, vias 2 -> 6
- net /ECB_D4: track 187.1 -> 147.4 mm, vias 3 -> 2
- net /ECB_A9: track 186.8 -> 149.0 mm, vias 2 -> 5
- net /~{ECB_INT}: track 87.5 -> 123.8 mm, vias 0 -> 3
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