File: MECB_8088/MECB_8088_CPU/MECB_8088_CPU.kicad_sch (KiCad schematic)
At the start: 28 parts, among them J1 MECB_64AC, SW1 SW_DIP_PB, U1 ATF22V10C-15PU, U2 SST39SF040, U3 AS6C4008-55, U4 TC1232CPA, U5 74HCT573, U6 74HCT75, U7 8088-2, Y1 8 MHz

Commit message: v1.1 - fix for missing ECB_CLK signal
Connections:
- net ECB_CLK: now also U1.14 (I/O_1)
Changed lines of the file:
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@@
 		(title "Minimalist Europe Card Bus (MECB) 8088 Board")
 		(date "2025-05")
-		(rev "1.0")
+		(rev "1.1")
 		(comment 1 "For Minimalist Europe Card Bus (MECB). ")
 	)
@@
 	(wire
 		(pts
+			(xy 200.66 53.34) (xy 209.55 53.34)
+		)
+		(stroke
+			(width 0)
+			(type default)
+		)
+	)
+	(wire
+		(pts
 			(xy 120.65 35.56) (xy 167.64 35.56)
 		)
@@
 		(effects
 			(font
+				(size 1.27 1.27)
+			)
+			(justify left bottom)
+		)
+	)
+	(label "ECB_CLK"
+		(at 200.66 53.34 0)
+		(effects
+			(font

Commit message: v1.1 8088 board
Parts:
- removed R1, R2, R3: 4K7, Resistor_THT:R_Axial_DIN0309_L9.0mm_D3.2mm_P12.70mm_Horizontal, symbol Device:R
- added J2: CLK_SEL, Connector_IDC:IDC-Header_2x03_P2.54mm_Vertical, symbol Connector_Generic:Conn_02x03_Odd_Even
- added RN2: 4K7, Resistor_THT:R_Array_SIP9, symbol Device:R_Network08_US
- RN1: value 10K -> 4K7
Connections:
- net RESET is gone; now on net HOLD: U1.8 (IN_6), U4.5 (RST), U5.1 (OE), U7.21 (RESET)
- net ~{M} is gone; now on net ~{ECB_MREQ}: U1.2 (IN_1), U7.28 (IO/~{M})
- net +5V: now also RN2.1 (common)
- net ECB_CLK: now also J2.2 (Pin_2), J2.4 (Pin_4), J2.6 (Pin_6); no longer U1.14 (I/O_1)
- net HOLD: no longer U1.15 (I/O_2)
- net INT: now also U1.18 (I/O_5); no longer U1.16 (I/O_3)
- net NMI: now also U1.19 (I/O_6); no longer U1.17 (I/O_4)
- net ~{CS_RAM}: now also U1.22 (I/O_9); no longer U1.21 (I/O_8)
- net ~{CS_ROM}: now also U1.23 (I/O_10); no longer U1.22 (I/O_9)
- net ~{ECB_INT}: now also RN2.3 (R2)
- net ~{ECB_IORQ}: now also U1.21 (I/O_8); no longer U1.20 (I/O_7)
- net ~{ECB_MREQ}: no longer U1.19 (I/O_6)
- net ~{ECB_NMI}: now also RN2.2 (R1)
- net ~{ECB_RESET}: now also U1.20 (I/O_7); no longer U1.18 (I/O_5)
- net ~{TEST}: now also RN2.4 (R3); no longer U1.23 (I/O_10)
- net at JP2.3 (B): now also RN2.9 (R8)
- net ~{SS0}: now reaches U7.34 (~{SSO})
- net ~{SS0}: now also U1.11 (IN_9)
- new net CLK/2: J2.1 (Pin_1), U1.17 (I/O_4)
- new net CLK/4: J2.3 (Pin_3), U1.16 (I/O_3)
- new net CLK/8: J2.5 (Pin_5), U1.15 (I/O_2)
Other:
- moved on the sheet: JP2, U6
