File: MECB_IDE/MECB_IDE.kicad_pcb (KiCad board)
At the start: 2 copper layers, 99.8 x 99.8 mm, 20 parts, among them J1 MECB_64AC, J2 Conn_02x20_Odd_Even, J3 Conn_02x22_Odd_Even, J4 Barrel_Jack_Switch, U1 ATF16V8, U2 82C55A, U3 74AHCT04

Commit message: Added note to remove pin 20 of 44 pin header
Other:
- board text added: "^Remove Pin"
Changed lines of the file:
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@@
 		(layer "Edge.Cuts")
+	)
+	(gr_text "^Remove\n Pin"
+		(at 192.5 92 90)
+		(layer "F.SilkS")
+		(effects
+			(font
+				(size 1 1)
+				(thickness 0.15)
+			)
+		)
 	)
 	(gr_text "MECB IDE Card v1.0\n"
