File: MECB_IO/MECB_IO.kicad_pcb (KiCad board)
At the start: 2 copper layers, 99.8 x 99.8 mm, 38 parts, among them J1 MECB_64AC, J2 Conn_02x10_Odd_Even, J3 Conn_01x03, SW1 SW_DIP_x08, U1 ATF22V10C-15PU, U2 74LS174, U3 DS1302+, U4 74LS245, U5 74LS374, Y1 32.768kHz

Commit message: V1.0 board should fix the RTC issue
Parts:
- removed REF**: LED_D3.0mm_Horizontal_O1.27mm_Z2.0mm, LED_THT:LED_D3.0mm_Horizontal_O1.27mm_Z2.0mm
- moved C3 15.5 mm to (135.0, 98.0)
- moved Y1 7.27 mm to (131.3, 89.7), turned to -90 degrees
- moved U3 2.38 mm to (134.9, 87.0)
Connections:
- R1 pad 1: /LED0 -> Net-(U5-O0)
- R1 pad 2: Net-(U5-O0) -> /LED0
- R2 pad 1: /LED1 -> Net-(U5-O1)
- R2 pad 2: Net-(U5-O1) -> /LED1
- R3 pad 1: /LED2 -> Net-(U5-O2)
- R3 pad 2: Net-(U5-O2) -> /LED2
- R5 pad 1: /LED4 -> Net-(U5-O4)
- R5 pad 2: Net-(U5-O4) -> /LED4
- R6 pad 1: /LED5 -> Net-(U5-O5)
- R6 pad 2: Net-(U5-O5) -> /LED5
- R7 pad 1: /LED6 -> Net-(U5-O6)
- R7 pad 2: Net-(U5-O6) -> /LED6
- R8 pad 1: /LED7 -> Net-(U5-O7)
- R8 pad 2: Net-(U5-O7) -> /LED7
- U1 pad 19: /RTC_WE -> /~{RTC_WE}
- Y1 pad 1: Net-(U3-X2) -> Net-(U3-X1)
- Y1 pad 2: Net-(U3-X1) -> Net-(U3-X2)
Routing:
- net /~{RTC_WE}: track 0.00 -> 68.3 mm
- net /LED4: track 93.9 -> 52.9 mm, vias 0 -> 1
- net +5V: track 339.9 -> 307.6 mm, vias 1 -> 2
- net /ECB_D4: track 80.3 -> 98.8 mm, vias 0 -> 2
- net /~{ECB_RESET}: track 150.8 -> 169.2 mm, vias 2 -> 1
- net Net-(U5-O1): track 51.4 -> 33.9 mm, vias 1 -> 0
- net /LED0: track 80.1 -> 63.6 mm
- net /ECB_D1: track 91.3 -> 75.3 mm
- net Net-(U5-O4): track 41.8 -> 26.3 mm, vias 1 -> 0
- net Net-(U5-O2): track 50.5 -> 35.4 mm
- net /ECB_D5: track 104.7 -> 90.2 mm, vias 3 -> 2
- net Net-(U5-O7): track 28.3 -> 14.3 mm
- net Net-(U5-O0): track 43.6 -> 29.7 mm, vias 1 -> 0
- net /LED7: track 58.5 -> 45.6 mm, vias 1 -> 0
- net Net-(U5-O5): track 28.1 -> 15.3 mm, vias 1 -> 0
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Other:
- board text added: "GND"
- board text added: "Reset"
- board text added: "VCC"
