File: MECB_SID/MECB_SID.kicad_pcb (KiCad board)
At the start: 2 copper layers, 99.8 x 99.8 mm, 45 parts, among them J1 MECB_64AC, J2 AudioJack3_SwitchTR, J3 MD205S-12B, J4 AudioJack3_SwitchTR, Q1 2N2222, Q2 2N2222, U1 ATF22V10C-15PU, U2 6581, U3 74LS374, U4 6581, Y1 1 MHz

Commit message: Pull WR signal down for v1.1 of board
Parts:
- removed JP2, JP3, JP4, JP5, JP6: Jumper_3_Bridged12, Connector_PinHeader_2.54mm:PinHeader_1x03_P2.54mm_Vertical
- added C19: 0.1uF, Capacitor_THT:C_Disc_D5.0mm_W2.5mm_P5.00mm, F.Cu at (125.0, 73.5)
- added U5: 74LS374, Package_DIP:DIP-20_W7.62mm_Socket_LongPads, F.Cu at (128.4, 78.5)
- U1: value ATF22V10C-15PU -> ATF16V8; footprint Package_DIP:DIP-24_W7.62mm_Socket_LongPads -> Package_DIP:DIP-20_W7.62mm_Socket_LongPads
- moved JP1 9.71 mm to (129.5, 68.0)
- moved U1 3.04 mm to (112.9, 65.5)
Connections:
- J1 pad A18: /ECB_A14 -> unconnected-(J1-A14-PadA18)
- J1 pad A20: /~{ECB_M1} -> unconnected-(J1-~{M1}-PadA20)
- J1 pad A29: /ECB_A13 -> unconnected-(J1-A13-PadA29)
- J1 pad A30: /ECB_A9 -> unconnected-(J1-A9-PadA30)
- J1 pad C17: /ECB_A11 -> unconnected-(J1-A11-PadC17)
- J1 pad C18: /ECB_A10 -> unconnected-(J1-A10-PadC18)
- J1 pad C20: /~{ECB_NMI} -> unconnected-(J1-~{NMI}-PadC20)
- J1 pad C21: /~{ECB_INT} -> unconnected-(J1-~{INT}-PadC21)
- J1 pad C27: /ECB_A12 -> unconnected-(J1-A12-PadC27)
- J1 pad C28: /ECB_A15 -> unconnected-(J1-A15-PadC28)
- J1 pad C30: /~{ECB_MREQ} -> unconnected-(J1-~{MREQ}-PadC30)
- J1 pad C8: /ECB_A8 -> unconnected-(J1-A8-PadC8)
- U1 pad 1: /ECB_CLK -> /~{ECB_IORQ}
- U1 pad 10: /ECB_A2 -> GND
- U1 pad 11: /ECB_A3 -> /ECB_A6
- U1 pad 12: GND -> /ECB_A7
- U1 pad 13: /ECB_A4 -> unconnected-(U1-IO7-Pad13)
- U1 pad 14: /ECB_A5 -> unconnected-(U1-IO6-Pad14)
- U1 pad 15: /ECB_A6 -> unconnected-(U1-IO5-Pad15)
- U1 pad 16: /ECB_A7 -> unconnected-(U1-IO4-Pad16)
- U1 pad 17: /~{IO_WR} -> unconnected-(U1-IO3-Pad17)
- U1 pad 18: unconnected-(U1-I/O_5-Pad18) -> /~{SID_ADDR}
- U1 pad 19: unconnected-(U1-I/O_6-Pad19) -> /~{SID_DATA}
- U1 pad 2: /RTC_IN -> /~{ECB_RD}
- U1 pad 20: unconnected-(U1-I/O_7-Pad20) -> +5V
- U1 pad 3: /~{ECB_IORQ} -> /~{ECB_WR}
- U1 pad 4: /~{ECB_RD} -> /ECB_A0
- U1 pad 5: /~{ECB_WR} -> /ECB_A1
- U1 pad 6: /~{ECB_M1} -> /ECB_A2
- U1 pad 7: /~{ECB_RESET} -> /ECB_A3
- U1 pad 8: /ECB_A0 -> /ECB_A4
- U1 pad 9: /ECB_A1 -> /ECB_A5
- U2 pad 10: /SID_A1 -> /L_A1
- U2 pad 11: /SID_A2 -> /L_A2
- U2 pad 12: /SID_A3 -> /L_A3
- U2 pad 13: /SID_A4 -> /L_A4
- U2 pad 15: /ECB_D0 -> /L_D0
- U2 pad 16: /ECB_D1 -> /L_D1
- U2 pad 17: /ECB_D2 -> /L_D2
- U2 pad 18: /ECB_D3 -> /L_D3
- U2 pad 19: /ECB_D4 -> /L_D4
- U2 pad 20: /ECB_D5 -> /L_D5
- U2 pad 21: /ECB_D6 -> /L_D6
- U2 pad 22: /ECB_D7 -> /L_D7
- U2 pad 7: /~{ECB_WR} -> GND
- U2 pad 9: /SID_A0 -> /L_A0
- U3 pad 16: unconnected-(U3-O6-Pad16) -> /~{SID_CS1}
- U3 pad 19: unconnected-(U3-O7-Pad19) -> /~{SID_CS2}
- U4 pad 10: /SID_A1 -> /L_A1
- U4 pad 11: /SID_A2 -> /L_A2
- U4 pad 12: /SID_A3 -> /L_A3
- U4 pad 13: /SID_A4 -> /L_A4
- U4 pad 15: /ECB_D0 -> /L_D0
- U4 pad 16: /ECB_D1 -> /L_D1
- U4 pad 17: /ECB_D2 -> /L_D2
- U4 pad 18: /ECB_D3 -> /L_D3
- U4 pad 19: /ECB_D4 -> /L_D4
- U4 pad 20: /ECB_D5 -> /L_D5
- U4 pad 21: /ECB_D6 -> /L_D6
- U4 pad 22: /ECB_D7 -> /L_D7
- U4 pad 7: /~{ECB_WR} -> GND
- U4 pad 9: /SID_A0 -> /L_A0
Routing:
- net /L_D0: track 0.00 -> 98.3 mm, vias 0 -> 2
- net /L_D1: track 0.00 -> 92.1 mm, vias 0 -> 2
- net /L_D2: track 0.00 -> 88.6 mm, vias 0 -> 1
- net /L_D3: track 0.00 -> 87.0 mm, vias 0 -> 1
- net GND: track 365.8 -> 451.1 mm
- net /~{ECB_WR}: track 96.3 -> 15.4 mm, vias 1 -> 0
- net /L_D4: track 0.00 -> 79.0 mm
- net /ECB_D0: track 144.5 -> 67.3 mm, vias 3 -> 2
- net /SID_A4: track 75.3 -> 0.00 mm, vias 1 -> 0
- net /L_D7: track 0.00 -> 75.1 mm
- net /L_D5: track 0.00 -> 73.4 mm, vias 0 -> 1
- net /L_D6: track 0.00 -> 73.1 mm, vias 0 -> 1
- net /SID_A3: track 71.2 -> 0.00 mm
- net /ECB_D1: track 126.3 -> 55.8 mm
- net /SID_A1: track 67.2 -> 0.00 mm, vias 2 -> 0
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Other:
- board text added: "MECB SID v1.1"
- board text removed: "MECB SID v0.1"
