File: MECB_SID/MECB_SID.kicad_sch (KiCad schematic)
At the start: 45 parts, among them J1 MECB_64AC, J2 AudioJack3_SwitchTR, J3 MD205S-12B, J4 AudioJack3_SwitchTR, Q1 2N2222, Q2 2N2222, U1 ATF22V10C-15PU, U2 6581, U3 74LS374, U4 6581, Y1 1 MHz

Commit message: Pull WR signal down for v1.1 of board
Parts:
- removed JP2, JP3, JP4, JP5, JP6: Jumper_3_Bridged12, Connector_PinHeader_2.54mm:PinHeader_1x03_P2.54mm_Vertical, symbol Jumper:Jumper_3_Bridged12
- removed U1: ATF22V10C-15PU, Package_DIP:DIP-24_W7.62mm_Socket_LongPads, symbol SamacSys_Parts:ATF22V10C-15PU
- added C19: 0.1uF, Capacitor_THT:C_Disc_D5.0mm_W2.5mm_P5.00mm, symbol Device:C
- added U1: ATF16V8, Package_DIP:DIP-20_W7.62mm_Socket_LongPads, symbol Custom:ATF16V8
- added U5: 74LS374, Package_DIP:DIP-20_W7.62mm_Socket_LongPads, symbol 74xx:74LS374
Connections:
- net SID_A0 is gone; now on net L_A0: U2.9 (A0), U4.9 (A0)
- net SID_A1 is gone; now on net L_A1: U2.10 (A1), U4.10 (A1)
- net SID_A2 is gone; now on net L_A2: U2.11 (A2), U4.11 (A2)
- net SID_A3 is gone; now on net L_A3: U2.12 (A3), U4.12 (A3)
- net SID_A4 is gone; now on net L_A4: U2.13 (A4), U4.13 (A4)
- net +5V: now also C19.2, U1.20 (VCC), U5.20 (VCC)
- net ECB_A0: now also U1.4 (I4)
- net ECB_A1: now also U1.5 (I5)
- net ECB_A2: now also U1.6 (I6)
- net ECB_A3: now also U1.7 (I7)
- net ECB_A4: now also U1.8 (I8)
- net ECB_A5: now also U1.9 (I9)
- net ECB_A6: now also U1.11 (I10/~{OE})
- net ECB_A7: now also U1.12 (IO8)
- net ECB_D0: now also U5.3 (D0); no longer U2.15 (D0), U4.15 (D0)
- net ECB_D1: now also U5.4 (D1); no longer U2.16 (D1), U4.16 (D1)
- net ECB_D2: now also U5.7 (D2); no longer U2.17 (D2), U4.17 (D2)
- net ECB_D3: now also U5.8 (D3); no longer U2.18 (D3), U4.18 (D3)
- net ECB_D4: now also U5.13 (D4); no longer U2.19 (D4), U4.19 (D4)
- net ECB_D5: now also U5.14 (D5); no longer U2.20 (D5), U4.20 (D5)
- net ECB_D6: now also U5.17 (D6); no longer U2.21 (D6), U4.21 (D6)
- net ECB_D7: now also U5.18 (D7); no longer U2.22 (D7), U4.22 (D7)
- net GND: now also U2.7 (R/~{W}), U4.7 (R/~{W}), C19.1, U1.10 (GND), U5.1 (OE), U5.10 (GND)
- net ~{ECB_IORQ}: now also U1.1 (I1/CLK)
- net ~{ECB_RD}: now also U1.2 (I2)
- net ~{ECB_WR}: now also U1.3 (I3); no longer U2.7 (R/~{W}), U4.7 (R/~{W})
- net ~{SID_ADDR}: now also U1.18 (IO2)
- net ~{SID_CS1}: now also U3.16 (O6)
- net ~{SID_CS2}: now also U3.19 (O7)
- net ECB_A10: no longer names the net of J1.C18 (A10)
- net ECB_A11: no longer names the net of J1.C17 (A11)
- net ECB_A12: no longer names the net of J1.C27 (A12)
- net ECB_A13: no longer names the net of J1.A29 (A13)
- net ECB_A14: no longer names the net of J1.A18 (A14)
- net ECB_A15: no longer names the net of J1.C28 (A15)
- net ECB_A8: no longer names the net of J1.C8 (A8)
- net ECB_A9: no longer names the net of J1.A30 (A9)
- net ~{ECB_INT}: no longer names the net of J1.C21 (~{INT})
- net ~{ECB_M1}: no longer names the net of J1.A20 (~{M1})
- net ~{ECB_MREQ}: no longer names the net of J1.C30 (~{MREQ})
- net ~{ECB_NMI}: no longer names the net of J1.C20 (~{NMI})
- new net L_D0: U2.15 (D0), U4.15 (D0), U5.2 (O0)
- new net L_D1: U2.16 (D1), U4.16 (D1), U5.5 (O1)
- new net L_D2: U2.17 (D2), U4.17 (D2), U5.6 (O2)
- new net L_D3: U2.18 (D3), U4.18 (D3), U5.9 (O3)
- new net L_D4: U2.19 (D4), U4.19 (D4), U5.12 (O4)
- new net L_D5: U2.20 (D5), U4.20 (D5), U5.15 (O5)
- new net L_D6: U2.21 (D6), U4.21 (D6), U5.16 (O6)
- new net L_D7: U2.22 (D7), U4.22 (D7), U5.19 (O7)
- new net ~{SID_DATA}: U1.19 (IO1), U5.11 (Cp)
- no-connect marks 29 -> 46
